File: VLF4_PCB.kicad_sch (KiCad schematic)
At the start: 8 parts, among them J1 Conn_02x10_Odd_Even, J2 Conn_02x10_Odd_Even

Commit message: r2 don
Parts:
- renumbered C42 to C51, C42 to C52, C42 to C53, C42 to C54, C42 to C55, C42 to C56
Connections:
- net Base Board/BLUE_LED_CTRL: now also J1.11 (Pin_11); no longer J1.9 (Pin_9)
- net Base Board/GPS_PPS: now also J1.13 (Pin_13); no longer J1.10 (Pin_10)
- net Base Board/GPS_RX: now also J1.10 (Pin_10); no longer J1.16 (Pin_16)
- net Base Board/GPS_TX: now also J1.8 (Pin_8); no longer J1.18 (Pin_18)
- net Base Board/GPS_nRST: now also J1.5 (Pin_5); no longer J1.3 (Pin_3)
- net Base Board/GREEN_LED_CTRL: now also J1.9 (Pin_9); no longer J1.13 (Pin_13)
- net Base Board/LORA_BUSY: now also J1.16 (Pin_16); no longer J1.11 (Pin_11)
- net Base Board/LORA_CS: now also J1.12 (Pin_12); no longer J1.8 (Pin_8)
- net Base Board/LORA_DIO1: now also J1.19 (Pin_19); no longer J1.12 (Pin_12)
- net Base Board/LORA_DIO2: now also J1.3 (Pin_3); no longer J1.7 (Pin_7)
- net Base Board/LORA_MISO: now also J1.18 (Pin_18); no longer J1.19 (Pin_19)
- net Base Board/LORA_RXEN: now also J1.7 (Pin_7); no longer J1.15 (Pin_15)
- net Base Board/LORA_SCK: now also J1.15 (Pin_15); no longer J1.17 (Pin_17)
- net Base Board/LORA_TXEN: now also J1.6 (Pin_6); no longer J1.14 (Pin_14)
- net Base Board/LORA_nRST: now also J1.14 (Pin_14); no longer J1.6 (Pin_6)
- net Base Board/RED_LED_CTRL: now also J1.17 (Pin_17); no longer J1.5 (Pin_5)
- net Extension Board/BLUE_LED_CTRL: now also J2.11 (Pin_11); no longer J2.9 (Pin_9)
- net Extension Board/GPS_PPS: now also J2.13 (Pin_13); no longer J2.10 (Pin_10)
- net Extension Board/GPS_RX: now also J2.10 (Pin_10); no longer J2.16 (Pin_16)
- net Extension Board/GPS_TX: now also J2.8 (Pin_8); no longer J2.18 (Pin_18)
- net Extension Board/GPS_nRST: now also J2.5 (Pin_5); no longer J2.3 (Pin_3)
- net Extension Board/GREEN_LED_CTRL: now also J2.9 (Pin_9); no longer J2.13 (Pin_13)
- net Extension Board/LORA_BUSY: now also J2.16 (Pin_16); no longer J2.11 (Pin_11)
- net Extension Board/LORA_CS: now also J2.12 (Pin_12); no longer J2.8 (Pin_8)
- net Extension Board/LORA_DIO1: now also J2.19 (Pin_19); no longer J2.12 (Pin_12)
- net Extension Board/LORA_DIO2: now also J2.3 (Pin_3); no longer J2.7 (Pin_7)
- net Extension Board/LORA_MISO: now also J2.18 (Pin_18); no longer J2.19 (Pin_19)
- net Extension Board/LORA_RXEN: now also J2.7 (Pin_7); no longer J2.15 (Pin_15)
- net Extension Board/LORA_SCK: now also J2.15 (Pin_15); no longer J2.17 (Pin_17)
- net Extension Board/LORA_TXEN: now also J2.6 (Pin_6); no longer J2.14 (Pin_14)
- net Extension Board/LORA_nRST: now also J2.14 (Pin_14); no longer J2.6 (Pin_6)
- net Extension Board/RED_LED_CTRL: now also J2.17 (Pin_17); no longer J2.5 (Pin_5)
