File: base_board.kicad_sch (KiCad schematic)
At the start: 10 parts

Commit message: r2 don
Other:
- sheet Peripherals ports: added MAG1_SCL, MAG1_SDA; removed MAG_SCL, MAG_SDA
- sheet STM ports: added MAG1_SCL, MAG1_SDA; removed MAG_SCL, MAG_SDA
- note added: "I2C4"
- note added: "UART8"
- note added: "USART3"
