File: extension_board.kicad_sch (KiCad schematic)
At the start: 28 parts, among them Q18 2N7002, Q19 2N7002, Q20 2N7002, U10 L80RE, U11 E22-900M30S

Commit message: r2 don
Parts:
- renumbered H1 to H5, H2 to H6, H3 to H7, H4 to H8
Connections:
- net GPS_RX: now also U10.2 (TXD1); no longer U10.1 (RXD1)
- net GPS_TX: now also U10.1 (RXD1); no longer U10.2 (TXD1)
Other:
- note added: "USART2"
