File: peripherals.kicad_sch (KiCad schematic)
At the start: 37 parts, among them Q16 MMBT5551_C2145, Q17 MMBT5551_C2145, U12 TJA1043TK/1Y, U4 W25Q512JVFIQ, U5 MS560702BA03-50, U6 H3LIS100DLTR, U7 MMC5603NJ, U8 LSM6DSMTR

Commit message: r2 don
Parts:
- removed BUZZER2: MLT-9032, Rocketry:BUZ-SMD_MLT-9032, symbol Rocketry:MLT-9032
- removed D4: B5819W_C8598, Rocketry:SOD-123_L2.7-W1.6-LS3.7-RD-1, symbol Rocketry:B5819W_C8598
- removed Q17: MMBT5551_C2145, Rocketry:SOT-23-3_L2.9-W1.3-P1.90-LS2.4-BR, symbol Rocketry:MMBT5551_C2145
- removed R24: 330R, Resistor_SMD:R_0402_1005Metric, symbol Device:R
Connections:
- net MAG_SCL renamed MAG1_SCL
- net MAG_SDA renamed MAG1_SDA
Other:
- note added: "I2C1"
- note added: "SPI1"
- note added: "SPI3"
- note added: "SPI4"
- note added: "SPI6"
- moved on the sheet: C13, C14, C15, C16, C50, U7, U8
