File: pyro.kicad_sch (KiCad schematic)
At the start: 26 parts, among them Q10 AP25P06K, Q11 CJ3407, Q12 CJ3407, Q13 MMBT5551_C2145, Q14 AP25P06K, Q15 CJ3407, Q3 CJ3407, Q4 AP25P06K, Q5 CJ3407, Q6 MMBT5551_C2145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

Commit message: r2 don
Parts:
- R14, R18, R22: value 33K -> 100K
- renumbered J_EXT1 to J_PYRO1
