File: stm.kicad_sch (KiCad schematic)
At the start: 20 parts, among them U9 STM32H723VGHx, X1 X322516MLB4SI

Commit message: r2 don
Parts:
- added JP3: SolderJumper_2_Open, Jumper:SolderJumper-2_P1.3mm_Open_TrianglePad1.0x1.5mm, symbol Jumper:SolderJumper_2_Open
- added RBOOT1: 10K, Resistor_SMD:R_0402_1005Metric, symbol Device:R
- renumbered C3 to C57
Connections:
- net MAG_SCL is gone; now on net GPS_PPS: U9.K10 (PD12)
- net MAG_SDA is gone; now on net LORA_BUSY: U9.J10 (PD13)
- net 3V3: now also JP3.1 (A)
- net 5V_EN: now also U9.B3 (PE3); no longer U9.J9 (PD9)
- net ACC_CS: now also U9.H2 (PA1); no longer U9.B7 (PD2)
- net ACC_MISO: now also U9.J3 (PA6); no longer U9.A6 (PB4(NJTRST))
- net ACC_MOSI: now also U9.K3 (PA7); no longer U9.D6 (PD7)
- net ACC_SCL: now also U9.H3 (PA5); no longer U9.A7 (PB3(JTDO)
- net ARM_DETECT: now also U9.G9 (PD11); no longer U9.K4 (PB1)
- net BARO_CLK: now also U9.A7 (PB3(JTDO); no longer U9.J7 (PB10)
- net BARO_CS: now also U9.A1 (PC14); no longer U9.D10 (PA10)
- net BARO_MISO: now also U9.A6 (PB4(NJTRST)); no longer U9.H10 (PB14)
- net BARO_MOSI: now also U9.C5 (PB5); no longer U9.G10 (PB15)
- net BAT_V_M: now also U9.F1 (PC0); no longer U9.J4 (PB0)
- net BLUE_LED_CTRL: now also U9.K8 (PB12); no longer U9.C4 (PE1)
- net BUZZER_CTRL: now also U9.G2 (PA0); no longer U9.A5 (PB7)
- net CAN_EN: now also U9.C7 (PD3); no longer U9.K7 (PB11)
- net CAN_ERR_N: now also U9.B7 (PD2); no longer U9.D7 (PD4)
- net CAN_RX: now also U9.D8 (PD0); no longer U9.K8 (PB12)
- net CAN_STB_N: now also U9.B6 (PD5); no longer U9.J6 (PE12)
- net CAN_TX: now also U9.E8 (PD1); no longer U9.J8 (PB13)
- net CURR_M: now also U9.F3 (PC3_C); no longer U9.H4 (PC5)
- net CURR_REF: now also U9.F2 (PC1); no longer U9.G4 (PC4)
- net EXT_1_UART_RX: now also U9.K7 (PB11); no longer U9.J2 (PA2)
- net EXT_1_UART_TX: now also U9.J7 (PB10); no longer U9.K2 (PA3)
- net EXT_2_I2C_SCL: now also U9.B5 (PB6); no longer U9.D9 (PA8)
- net EXT_2_I2C_SDA: now also U9.A5 (PB7); no longer U9.E9 (PC9)
- net EXT_2_UART_RX: now also U9.D4 (PE0); no longer U9.E10 (PC7)
- net EXT_2_UART_TX: now also U9.C4 (PE1); no longer U9.F10 (PC6)
- net FLASH_CLK: now also U9.J6 (PE12); no longer U9.A3 (PE2)
- net FLASH_CS: now also U9.H7 (PE15); no longer U9.F2 (PC1)
- net FLASH_MISO: now also U9.K6 (PE13); no longer U9.D3 (PE5)
- net FLASH_MOSI: now also U9.G7 (PE14); no longer U9.E3 (PE6)
- net FLASH_nRESET: now also U9.J9 (PD9); no longer U9.B6 (PD5)
- net GND: now also U9.F9 (PC8), U9.H5 (PE7), U9.H6 (PE11), RBOOT1.2; no longer U9.D5 (BOOT0)
- net GPS_PPS: no longer U9.C5 (PB5)
- net GPS_RX: now also U9.K2 (PA3); no longer U9.G2 (PA0)
- net GPS_TX: now also U9.J2 (PA2); no longer U9.H2 (PA1)
- net GPS_nRST: now also U9.K5 (PE9); no longer U9.B5 (PB6)
- net GREEN_LED_CTRL: now also U9.G4 (PC4); no longer U9.C3 (PE4)
- net IMU_CS: now also U9.A2 (PC13); no longer U9.A8 (PA15(JTDI))
- net LORA_BUSY: no longer U9.A1 (PC14)
- net LORA_CS: now also U9.J4 (PB0); no longer U9.B3 (PE3)
- net LORA_DIO1: now also U9.G8 (PD15); no longer U9.B1 (PC15)
- net LORA_DIO2: now also U9.K4 (PB1); no longer U9.B4 (PB8)
- net LORA_MISO: now also U9.H10 (PB14); no longer U9.J3 (PA6)
- net LORA_MOSI: now also U9.G10 (PB15); no longer U9.K3 (PA7)
- net LORA_RXEN: now also U9.H4 (PC5); no longer U9.F1 (PC0)
- net LORA_SCK: now also U9.J8 (PB13); no longer U9.H3 (PA5)
- net LORA_TXEN: now also U9.H8 (PD14); no longer U9.E2 (PC2_C)
- net LORA_nRST: now also U9.J5 (PE8); no longer U9.A2 (PC13)
- net PYRO1_CONT: now also U9.F10 (PC6); no longer U9.K6 (PE13)
- net PYRO1_CTRL: now also U9.E9 (PC9); no longer U9.H7 (PE15)
- net PYRO2_CONT: now also U9.D10 (PA10); no longer U9.H9 (PD10)
- net PYRO2_CTRL: now also U9.E10 (PC7); no longer U9.H8 (PD14)
- net PYRO3_CONT: now also U9.D9 (PA8); no longer U9.G9 (PD11)
- net PYRO3_CTRL: now also U9.D7 (PD4); no longer U9.F9 (PC8)
- net RED_LED_CTRL: now also U9.H9 (PD10); no longer U9.A4 (PB9)
- net VDDA: now reaches C24.1, C25.1, L3.1, U9.H1 (VDDA)
- new net: JP3.2 (B), RBOOT1.1, U9.D5 (BOOT0)
- new net MAG1_SCL: U9.B4 (PB8)
- new net MAG1_SDA: U9.A4 (PB9)
Other:
- note added: "TIM2_CH1"
- moved on the sheet: C32, C33, X1
Changed lines of the file:
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@@
-(kicad_sch (version 20230121) (generator eeschema)
-  (paper "A4")
+(kicad_sch
+	(version 20231120)
+	(generator "eeschema")
+	(generator_version "8.0")
+	(paper "A4")
